File: FourThirdsEye.kicad_sch (KiCad schematic)
At the start: 116 parts, among them J1 QWIIC_CONNECTORJS-1MM, J3 Conn_Coaxial, J4 Conn_Coaxial, J5 Conn_Coaxial, J9 Conn_01x22_Female, U1 AP3418KTR-G1, U2 IMX294, U3 LP5907MFX-1.8, U4 TPS7A90, U5 ECS-2520MV-240-DN-TR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

Commit message: upload V2.1 files and Cmount adaptor 3D model
Parts:
- removed J1: QWIIC_CONNECTORJS-1MM, Connector_JST:JST_SH_BM04B-SRSS-TB_1x04-1MP_P1.00mm_Vertical, symbol SparkFun-Connectors:QWIIC_CONNECTORJS-1MM
- removed J5: Conn_Coaxial, U.FL_Hirose_U.FL-R-SMT-1_Vertical, symbol Connector:Conn_Coaxial
- removed R9: DNP, Resistor_SMD:R_0402_1005Metric, symbol Device:R
- added C73: 100nF, Capacitor_SMD:C_0402_1005Metric, symbol Device:C
- added C74: 10nF, Capacitor_SMD:C_0402_1005Metric, symbol Device:C
- added C75: 1uF, Capacitor_SMD:C_0402_1005Metric, symbol Device:C
- added J1: Conn_01x04_Shielded, Connector_JST:JST_SH_BM04B-SRSS-TB_1x04-1MP_P1.00mm_Vertical, symbol Connector_Generic_Shielded:Conn_01x04_Shielded
- added U8: ICM-42688-P, footprints:PQFN50P300X250X97-14N, symbol ICM-42688-P:ICM-42688-P
- C67: value 10nF -> 1uF
- J9: footprint footprints:XF2M22151A -> footprints:TF3822S05SV830
Connections:
- net +1V8: now also C73.1, C74.1, C75.1, U8.12 (AP_CS), U8.5 (VDDIO), U8.8 (VDD)
- net +3V3: now also J1.2 (Pin_2)
- net CAM1_CLK_N: now also FL3.2; no longer FL3.3
- net CAM1_CLK_P: now also FL3.3; no longer FL3.2
- net CAM1_D0_N: now also FL1.2; no longer FL1.3
- net CAM1_D0_P: now also FL1.3; no longer FL1.2
- net CAM1_D1_N: now also FL2.2; no longer FL2.3
- net CAM1_D1_P: now also FL2.3; no longer FL2.2
- net CAM1_D2_N: now also FL4.2; no longer FL4.3
- net CAM1_D2_P: now also FL4.3; no longer FL4.2
- net CAM1_D3_N: now also FL5.2; no longer FL5.3
- net CAM1_D3_P: now also FL5.3; no longer FL5.2
- net CAM_CLK_N: now also FL3.1; no longer FL3.4
- net CAM_CLK_P: now also FL3.4; no longer FL3.1
- net CAM_D0_N: now also FL1.1; no longer FL1.4
- net CAM_D0_P: now also FL1.4; no longer FL1.1
- net CAM_D1_N: now also FL2.1; no longer FL2.4
- net CAM_D1_P: now also FL2.4; no longer FL2.1
- net CAM_D2_N: now also FL4.1; no longer FL4.4
- net CAM_D2_P: now also FL4.4; no longer FL4.1
- net CAM_D3_N: now also FL5.1; no longer FL5.4
- net CAM_D3_P: now also FL5.4; no longer FL5.1
- net GND: now also C73.2, C74.2, C75.2, J1.1 (Pin_1), J1.MP (Shield), U8.1 (AP_SDO/AP_AD0), U8.10 (RESV_10), U8.11 (RESV_11), U8.2 (RESV_2), U8.3 (RESV_3), U8.6 (GND), U8.7 (RESV_7)
- net SCL_1V8: now also U8.13 (AP_SCL/AP_SCLK)
- net SCL_3V3: now also J1.4 (Pin_4)
- net SDA_1V8: now also U8.14 (AP_SDA/AP_SDIO/AP_SDI)
- net SDA_3V3: now also J1.3 (Pin_3)
- net XVS: now also U8.9 (INT2/FSYNC/CLKIN)
Other:
- note added: "I2C ADDR: 0x68"
- note added: "IMU"
- note added: "QWIIC"
- moved on the sheet: C71, C72, FL1, FL2, FL3, FL4, FL5, H1, H2, H3, H4, J3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
